File: solar-curve-tracer.kicad_sch (KiCad schematic)
At the start: 5 parts, among them U1 TMP117NAIDRVR, U2 INA226

Commit message: schematic
Parts:
- added C1: C_Small, Capacitor_SMD:C_0603_1608Metric_Pad1.08x0.95mm_HandSolder, symbol Device:C_Small
- added C2, C3: 0.1uF, Capacitor_SMD:C_0603_1608Metric, symbol Device:C_Small
Connections:
- net GND: now also R1.2, SC1.2 (-), U1.2 (GND), U2.9 (Vin-), C2.2, C3.2
- net at R1.1, SC1.1 (+), U2.10 (Vin+): now also U2.8 (Vbus)
- net SDA: now reaches U2.4 (SDA)
- net SDA: now also U1.6 (SDA)
- net SCL: now reaches U2.5 (SCL)
- net SCL: now also U1.1 (SCL)
- net +3.3V: now reaches U2.6 (VS)
- net +3.3V: now also U1.5 (V+), C2.1, C3.1
- no-connect marks 0 -> 2
Other:
- moved on the sheet: U1

Commit message: schematic
Parts:
- removed C1: C_Small, Capacitor_SMD:C_0603_1608Metric_Pad1.08x0.95mm_HandSolder, symbol Device:C_Small
- removed U1: TMP117NAIDRVR, Package_SON:WSON-6-1EP_2x2mm_P0.65mm_EP1x1.6mm, symbol Sensor_Temperature:TMP117xxDRV
- added C4, C5, C6, C8: 0.1uF, Capacitor_SMD:C_0603_1608Metric, symbol Device:C_Small
- added C7: 56pF, Capacitor_SMD:C_0603_1608Metric, symbol Device:C_Small
- added Q1: IXTH64N10L2, Package_TO_SOT_THT:TO-247-3_Vertical, symbol Transistor_FET:IRFP4468PbF
- added R10, R9: 10K, Resistor_SMD:R_0805_2012Metric_Pad1.20x1.40mm_HandSolder, symbol Device:R_US
- added R3: 1m, Resistor_SMD:R_Shunt_Vishay_WSK2512_6332Metric_T1.19mm, symbol Device:R_Shunt_US
- added R4, R5: 1K, Resistor_SMD:R_0603_1608Metric_Pad0.98x0.95mm_HandSolder, symbol Device:R_US
- added R6, R7, R8: 15K, Resistor_SMD:R_0603_1608Metric_Pad0.98x0.95mm_HandSolder, symbol Device:R_US
- added U1: LT1806IS8#PBF, Package_SO:SOIC-8_3.9x4.9mm_P1.27mm, symbol Amplifier_Operational:LT1363
- added U3: LM2665M6, Package_TO_SOT_SMD:SOT-23-6, symbol Regulator_SwitchedCapacitor:LM2665M6
- added U4: ESP32-C3-DevKitM-1, RF_Module:ESP32-C3-DevKitM-1, symbol RF_Module:ESP32-C3-DevKitM-1
- added U5, U7, U8: TMP1075DGK, Package_SO:VSSOP-8_3x3mm_P0.65mm, symbol Sensor_Temperature:TMP1075DGK
- added U6: MAX5812MEUT+T, Package_TO_SOT_SMD:SOT-23-6_Handsoldering, symbol jannett_symbols:MAX5812MEUT+T
- added U9: INA226, Package_SO:HVSSOP-10-1EP_3x3mm_P0.5mm_EP1.83x1.89mm, symbol Sensor_Energy:INA226
- R2: value R_US -> 47
- U2: footprint Package_SO:VSSOP-10_3x3mm_P0.5mm -> Package_SO:HVSSOP-10-1EP_3x3mm_P0.5mm_EP1.83x1.89mm
Connections:
- net +3.3V: now also C4.1, C5.1, C6.1, C8.1, R6.2, U5.8 (V+), U6.1 (VDD), U7.8 (V+), U8.8 (V+), U9.6 (VS)
- net GND: now also U2.1 (A1), U2.2 (A0), C4.2, C5.2, C6.2, C8.2, R10.1, R3.4, R8.1, U1.4 (V-), U3.2 (GND), U4.1 (GND), U4.12 (GND), U4.15 (GND), U4.16 (GND), U4.19 (GND), U4.24 (GND), U4.27 (GND), U4.30 (GND), U4.6 (GND), U4.8 (GND), U5.4 (GND), U6.2 (VSS), U7.4 (GND), U8.4 (GND), U9.1 (A1), U9.2 (A0), U9.7 (GND)
- net SCL: now also U5.2 (SCL), U6.4 (SCL), U7.2 (SCL), U8.2 (SCL), U9.5 (SCL)
- net SDA: now also U5.1 (SDA), U6.3 (SDA), U7.1 (SDA), U8.1 (SDA), U9.4 (SDA)
- net at R2.1: now also C7.1, U1.6
- net at R2.2: now also Q1.1 (G)
- new net: R3.2, R4.2, U9.10 (Vin+)
- new net: R10.2, R9.1, U9.8 (Vbus)
- new net: R3.3, R5.2, U9.9 (Vin-)
- new net: U4.13 (5V), U4.14 (5V)
- new net: U4.2 (3V3), U4.3 (3V3)
- new net: R5.1, R7.2, U1.3 (+)
- new net: C7.2, R4.1, R8.2, U1.2 (-)
- new net: R7.1, U6.6 (VOUT)
- new net: Q1.3 (S), R3.1
- new net: R6.1, U1.1 (VOS), U8.3 (ALERT)
- new net: Q1.2 (D), R9.2
- no-connect marks 2 -> 5
Other:
- moved on the sheet: C2, C3, R1, R2, SC1, U2
